File: audio.kicad_sch (KiCad schematic)
At the start: 51 parts, among them J10 Earth, J4 NCJ6FA-H-0, J5 NCJ6FA-H-0, J6 Conn_01x04_Pin, J7 Earth, J8 NCJ6FA-H-0, J9 NCJ6FA-H-0, U5 THAT1246, U6 THAT1246, U7 THAT1646, U8 THAT1646

Commit message: merge libraries
Parts:
- S1: symbol LC2255EESP:LC2255EESP -> daisy-studio:LC2255EESP
- U5, U6: symbol triptech:THAT1246 -> daisy-studio:THAT1246
- U7, U8: symbol triptech:THAT1646 -> daisy-studio:THAT1646
Changed lines of the file:
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@@
 	)
 	(symbol
-		(lib_id "LC2255EESP:LC2255EESP")
+		(lib_id "daisy-studio:LC2255EESP")
 		(at 86.36 100.33 0)
 		(unit 1)
@@
 	(symbol
 		(lib_name "THAT1246_1")
-		(lib_id "triptech:THAT1246")
+		(lib_id "daisy-studio:THAT1246")
 		(at 58.42 107.95 0)
 		(unit 1)
@@
 	(symbol
 		(lib_name "THAT1646_1")
-		(lib_id "triptech:THAT1646")
+		(lib_id "daisy-studio:THAT1646")
 		(at 205.74 102.87 0)
 		(unit 1)
@@
 	(symbol
 		(lib_name "THAT1246_1")
-		(lib_id "triptech:THAT1246")
+		(lib_id "daisy-studio:THAT1246")
 		(at 58.42 45.72 0)
 		(unit 1)
@@
 	(symbol
 		(lib_name "THAT1646_1")
-		(lib_id "triptech:THAT1646")
+		(lib_id "daisy-studio:THAT1646")
 		(at 205.74 40.64 0)
 		(unit 1)

Commit message: fix lib refs
Parts:
- S1: footprint libs:LC2255EESP -> daisy-studio:LC2255EESP
Changed lines of the file:
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@@
 			)
 		)
-		(property "Footprint" "libs:LC2255EESP"
+		(property "Footprint" "daisy-studio:LC2255EESP"
 			(at 113.03 195.25 0)
 			(effects
