File: audio.kicad_sch (KiCad schematic)
At the start: 52 parts, among them J10 NCJ6FA-H-0, J9 NCJ6FA-H-0, Q1 2N3904, Q2 2N3904, Q3 2N3906, Q4 2N3906, U10 OPA1656ID, U11 LM2903, U8 THAT1246, U9 THAT1246

Commit message: All the testpoints
Parts:
- added TP10: RIP, symbol Connector:TestPoint
- added TP11: L-4dB, symbol Connector:TestPoint
- added TP12: R-4dB, symbol Connector:TestPoint
- added TP13: LGAIN, symbol Connector:TestPoint
- added TP14: RGAIN, symbol Connector:TestPoint
- added TP15: LWIPER, symbol Connector:TestPoint
- added TP16: RWIPER, symbol Connector:TestPoint
- added TP17: LCLIP, TestPoint:TestPoint_Pad_1.5x1.5mm, symbol Connector:TestPoint
- added TP18: RCLIP, TestPoint:TestPoint_Pad_1.5x1.5mm, symbol Connector:TestPoint
- added TP7: LIP, symbol Connector:TestPoint
- added TP8: LIN, symbol Connector:TestPoint
- added TP9: RIN, symbol Connector:TestPoint
- C26: renamed from C30; footprint (none) -> Capacitor_SMD:C_0805_2012Metric
- C27: renamed from C33; footprint (none) -> Capacitor_SMD:C_0805_2012Metric
- C28: renamed from C29; footprint (none) -> Capacitor_SMD:C_0805_2012Metric
- C29: renamed from C28; footprint (none) -> Capacitor_SMD:C_0805_2012Metric
- C30: renamed from C32; footprint (none) -> Capacitor_SMD:C_0805_2012Metric
- C31: renamed from C38; footprint (none) -> Capacitor_SMD:C_0805_2012Metric
- C32: renamed from C40; footprint (none) -> Capacitor_SMD:C_0805_2012Metric
- C33: renamed from C41; footprint (none) -> Capacitor_SMD:C_0805_2012Metric
- C34: renamed from C50; footprint (none) -> Capacitor_SMD:C_0805_2012Metric
- C35: renamed from C51; footprint (none) -> Capacitor_SMD:C_0805_2012Metric
- C36: renamed from C39; footprint (none) -> Capacitor_SMD:C_0805_2012Metric
- C37: renamed from C31; footprint (none) -> Capacitor_SMD:C_0805_2012Metric
- C38: renamed from C18; footprint (none) -> Capacitor_SMD:C_0805_2012Metric
- C39: renamed from C19; footprint (none) -> Capacitor_SMD:C_0805_2012Metric
- RV7: renamed from RV5; footprint (none) -> Potentiometer_THT:Potentiometer_Bourns_3296W_Vertical
- RV8: renamed from RV6; footprint (none) -> Potentiometer_THT:Potentiometer_Bourns_3296W_Vertical
- TP1: renamed from TP2; footprint (none) -> TestPoint:TestPoint_Pad_1.5x1.5mm
- TP2: renamed from TP1; footprint (none) -> TestPoint:TestPoint_Pad_1.5x1.5mm
- TP3: renamed from TP5; footprint (none) -> TestPoint:TestPoint_Pad_1.5x1.5mm
- TP4: renamed from TP6; footprint (none) -> TestPoint:TestPoint_Pad_1.5x1.5mm
- TP5: renamed from TP3; footprint (none) -> TestPoint:TestPoint_Pad_1.5x1.5mm
- TP6: renamed from TP4; footprint (none) -> TestPoint:TestPoint_Pad_1.5x1.5mm
- renumbered C34 to C40, C35 to C41, C36 to C42, C37 to C43, J9 to J12, J10 to J13, Q2 to Q1, Q1 to Q2, Q4 to Q3, Q3 to Q4, R19 to R23, R20 to R24, R21 to R25, R22 to R26, R23 to R27, R24 to R28, R25 to R29, R26 to R30, R27 to R31, R28 to R32, R29 to R33, R30 to R34, R31 to R35, R32 to R36, R33 to R37, R34 to R38, U8 to U10, U9 to U11, U10 to U8, U11 to U9
Connections:
- net CLIP_LED_K_L: now also TP17.1
- net CLIP_LED_K_R: now also TP18.1
- net IN_OPA_L: now also TP13.1
- net IN_OPA_R: now also TP14.1
- net IN_THRESH_L: no longer RV8.2, U9.5 (+)
- net IN_WIPER_L: now also TP15.1
- net IN_WIPER_R: now also TP16.1
- net at J13.3, J13.R, U11.2 (-): now also TP10.1
- net at J13.2, J13.T, U11.3 (+): now also TP9.1
- net at J12.2, J12.T, U10.3 (+): now also TP8.1
- net at J12.3, J12.R, U10.2 (-): now also TP7.1
- net at R23.1, U10.6: now also TP11.1
- net at R24.1, U11.6: now also TP12.1
- new net IN_THRESH_R: RV8.2, U9.5 (+)
Other:
- note removed: "To Seed"

Commit message: wip
Parts:
- renumbered TP7 to TP1, TP16 to TP10, TP1 to TP11, TP17 to TP12, TP2 to TP13, TP18 to TP14, TP3 to TP15, TP4 to TP16, TP5 to TP17, TP6 to TP18, TP8 to TP2, TP10 to TP3, TP9 to TP4, TP12 to TP5, TP11 to TP6, TP13 to TP7, TP14 to TP8, TP15 to TP9
Changed lines of the file:
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@@
 	(wire
 		(pts
-			(xy 238.76 64.77) (xy 238.76 66.04)
-		)
-		(stroke
-			(width 0)
-			(type default)
-		)
-	)
-	(wire
-		(pts
 			(xy 163.83 116.84) (xy 163.83 104.14)
 		)
@@
 	(wire
 		(pts
+			(xy 238.76 64.77) (xy 238.76 66.04)
+		)
+		(stroke
+			(width 0)
+			(type default)
+		)
+	)
+	(wire
+		(pts
 			(xy 48.26 158.75) (xy 52.07 158.75)
 		)
@@
 		(on_board yes)
 		(dnp no)
-		(property "Reference" "TP12"
+		(property "Reference" "TP5"
 			(at 60.452 114.554 0)
 			(effects
@@
 			(project "daisy-studio"
 				(path "/55cca6a8-30da-4c13-b2f2-a01401e2b54c/a1b2c3d4-7777-4000-8000-000000000007"
-					(reference "TP12")
+					(reference "TP5")
 					(unit 1)
 				)
@@
 		(on_board yes)
 		(dnp no)
-		(property "Reference" "TP18"
+		(property "Reference" "TP14"
 			(at 190.5 123.444 0)
 			(effects
@@
 			(project "daisy-studio"
 				(path "/55cca6a8-30da-4c13-b2f2-a01401e2b54c/a1b2c3d4-7777-4000-8000-000000000007"
-					(reference "TP18")
+					(reference "TP14")
 					(unit 1)
 				)
@@
 		(on_board yes)
 		(dnp no)
-		(property "Reference" "TP8"
+		(property "Reference" "TP2"
 			(at 40.132 53.594 0)
 			(effects
@@
 			(project "daisy-studio"
 				(path "/55cca6a8-30da-4c13-b2f2-a01401e2b54c/a1b2c3d4-7777-4000-8000-000000000007"
-					(reference "TP8")
+					(reference "TP2")
 					(unit 1)
 				)
@@
 		(on_board yes)
 		(dnp no)
-		(property "Reference" "TP9"
+		(property "Reference" "TP4"
 			(at 40.132 115.824 0)
 			(effects
@@
 			(project "daisy-studio"
 				(path "/55cca6a8-30da-4c13-b2f2-a01401e2b54c/a1b2c3d4-7777-4000-8000-000000000007"
-					(reference "TP9")
+					(reference "TP4")
 					(unit 1)
 				)
@@
 		(on_board yes)
 		(dnp no)
-		(property "Reference" "TP3"
+		(property "Reference" "TP15"
 			(at 223.52 116.078 0)
 			(effects
@@
 			(project "daisy-studio"
 				(path "/55cca6a8-30da-4c13-b2f2-a01401e2b54c/a1b2c3d4-7777-4000-8000-000000000007"
-					(reference "TP3")
+					(reference "TP15")
 					(unit 1)
 				)
@@
 		(on_board yes)
 		(dnp no)
-		(property "Reference" "TP13"
+		(property "Reference" "TP7"
 			(at 96.012 54.864 0)
 			(effects
@@
 			(project "daisy-studio"
 				(path "/55cca6a8-30da-4c13-b2f2-a01401e2b54c/a1b2c3d4-7777-4000-8000-000000000007"
-					(reference "TP13")
+					(reference "TP7")
 					(unit 1)
 				)
@@
 		(on_board yes)
 		(dnp no)
-		(property "Reference" "TP17"
+		(property "Reference" "TP12"
 			(at 190.5 61.214 0)
 			(effects
@@
 			(project "daisy-studio"
 				(path "/55cca6a8-30da-4c13-b2f2-a01401e2b54c/a1b2c3d4-7777-4000-8000-000000000007"
-					(reference "TP17")
+					(reference "TP12")
 					(unit 1)
 				)
@@
 		(on_board yes)
 		(dnp no)
-		(property "Reference" "TP7"
+		(property "Reference" "TP1"
 			(at 40.132 35.306 0)
 			(effects
@@
 			(project ""
 				(path "/55cca6a8-30da-4c13-b2f2-a01401e2b54c/a1b2c3d4-7777-4000-8000-000000000007"
-					(reference "TP7")
+					(reference "TP1")
 					(unit 1)
 				)
@@
 		(on_board yes)
 		(dnp no)
-		(property "Reference" "TP14"
+		(property "Reference" "TP8"
 			(at 96.012 117.094 0)
 			(effects
@@
 			(project "daisy-studio"
 				(path "/55cca6a8-30da-4c13-b2f2-a01401e2b54c/a1b2c3d4-7777-4000-8000-000000000007"
-					(reference "TP14")
+					(reference "TP8")
 					(unit 1)
 				)
@@
 		(on_board yes)
 		(dnp no)
-		(property "Reference" "TP1"
+		(property "Reference" "TP11"
 			(at 184.658 42.926 0)
 			(effects
@@
 			(project "daisy-studio"
 				(path "/55cca6a8-30da-4c13-b2f2-a01401e2b54c/a1b2c3d4-7777-4000-8000-000000000007"
-					(reference "TP1")
+					(reference "TP11")
 					(unit 1)
 				)
@@
 		(on_board yes)
 		(dnp no)
-		(property "Reference" "TP5"
+		(property "Reference" "TP17"
 			(at 224.79 39.878 0)
 			(effects
@@
 			(project "daisy-studio"
 				(path "/55cca6a8-30da-4c13-b2f2-a01401e2b54c/a1b2c3d4-7777-4000-8000-000000000007"
-					(reference "TP5")
+					(reference "TP17")
 					(unit 1)
 				)
@@
 		(on_board yes)
 		(dnp no)
-		(property "Reference" "TP16"
+		(property "Reference" "TP10"
 			(at 126.746 117.094 0)
 			(effects
@@
 			(project "daisy-studio"
 				(path "/55cca6a8-30da-4c13-b2f2-a01401e2b54c/a1b2c3d4-7777-4000-8000-000000000007"
-					(reference "TP16")
+					(reference "TP10")
 					(unit 1)
 				)
@@
 		(on_board yes)
 		(dnp no)
-		(property "Reference" "TP2"
+		(property "Reference" "TP13"
 			(at 184.658 105.156 0)
 			(effects
@@
 			(project "daisy-studio"
 				(path "/55cca6a8-30da-4c13-b2f2-a01401e2b54c/a1b2c3d4-7777-4000-8000-000000000007"
-					(reference "TP2")
+					(reference "TP13")
 					(unit 1)
 				)
@@
 		(on_board yes)
 		(dnp no)
-		(property "Reference" "TP4"
+		(property "Reference" "TP16"
 			(at 223.52 151.638 0)
 			(effects
@@
 			(project "daisy-studio"
 				(path "/55cca6a8-30da-4c13-b2f2-a01401e2b54c/a1b2c3d4-7777-4000-8000-000000000007"
-					(reference "TP4")
+					(reference "TP16")
 					(unit 1)
 				)
@@
 		(on_board yes)
 		(dnp no)
-		(property "Reference" "TP15"
+		(property "Reference" "TP9"
 			(at 126.746 54.864 0)
 			(effects
@@
 			(project "daisy-studio"
 				(path "/55cca6a8-30da-4c13-b2f2-a01401e2b54c/a1b2c3d4-7777-4000-8000-000000000007"
-					(reference "TP15")
+					(reference "TP9")
 					(unit 1)
 				)
@@
 		(on_board yes)
 		(dnp no)
-		(property "Reference" "TP11"
+		(property "Reference" "TP6"
 			(at 61.722 52.324 0)
 			(effects
@@
 			(project "daisy-studio"
 				(path "/55cca6a8-30da-4c13-b2f2-a01401e2b54c/a1b2c3d4-7777-4000-8000-000000000007"
-					(reference "TP11")
+					(reference "TP6")
 					(unit 1)
 				)
@@
 		(on_board yes)
 		(dnp no)
-		(property "Reference" "TP10"
+		(property "Reference" "TP3"
 			(at 40.132 97.536 0)
 			(effects
@@
 			(project "daisy-studio"
 				(path "/55cca6a8-30da-4c13-b2f2-a01401e2b54c/a1b2c3d4-7777-4000-8000-000000000007"
-					(reference "TP10")
+					(reference "TP3")
 					(unit 1)
 				)
@@
 		(on_board yes)
 		(dnp no)
-		(property "Reference" "TP6"
+		(property "Reference" "TP18"
 			(at 224.79 75.438 0)
 			(effects
@@
 			(project "daisy-studio"
 				(path "/55cca6a8-30da-4c13-b2f2-a01401e2b54c/a1b2c3d4-7777-4000-8000-000000000007"
-					(reference "TP6")
+					(reference "TP18")
 					(unit 1)
 				)
