File: daisy_seed.kicad_sch (KiCad schematic)
At the start: 21 parts, among them J2 GPIO Header, J3 Micro_SD_Card, U3 Daisy_Seed, U4 H11L1SM

Commit message: merge libraries
Parts:
- J_MIDI_IN_1, J_MIDI_OUT_1, J_MIDI_THRU1: symbol SDS-50J:SDS-50J -> daisy-studio:SDS-50J
- U3: footprint daisy:DAISY_SEED_SMT -> daisy-studio:DAISY_SEED_SMT; symbol Daisy-Boards:Daisy_Seed -> daisy-studio:Daisy_Seed
Changed lines of the file:
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@@
 	)
 	(symbol
-		(lib_id "Daisy-Boards:Daisy_Seed")
+		(lib_id "daisy-studio:Daisy_Seed")
 		(at 78.74 102.87 0)
 		(unit 1)
@@
 			)
 		)
-		(property "Footprint" "daisy:DAISY_SEED_SMT"
+		(property "Footprint" "daisy-studio:DAISY_SEED_SMT"
 			(at 83.82 135.89 0)
 			(effects
@@
 	)
 	(symbol
-		(lib_id "SDS-50J:SDS-50J")
+		(lib_id "daisy-studio:SDS-50J")
 		(at 248.92 109.22 0)
 		(unit 1)
@@
 	(symbol
 		(lib_name "SDS-50J_2")
-		(lib_id "SDS-50J:SDS-50J")
+		(lib_id "daisy-studio:SDS-50J")
 		(at 248.92 135.89 0)
 		(unit 1)
@@
 	)
 	(symbol
-		(lib_id "SDS-50J:SDS-50J")
+		(lib_id "daisy-studio:SDS-50J")
 		(at 331.47 125.73 0)
 		(unit 1)

Commit message: fix lib refs
Parts:
- J_MIDI_IN_1, J_MIDI_OUT_1, J_MIDI_THRU1: footprint libs:SDS50J -> daisy-studio:SDS50J
Changed lines of the file:
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@@
 			)
 		)
-		(property "Footprint" "libs:SDS50J"
+		(property "Footprint" "daisy-studio:SDS50J"
 			(at 267.97 204.14 0)
 			(effects
@@
 			)
 		)
-		(property "Footprint" "libs:SDS50J"
+		(property "Footprint" "daisy-studio:SDS50J"
 			(at 267.97 230.81 0)
 			(effects
@@
 			)
 		)
-		(property "Footprint" "libs:SDS50J"
+		(property "Footprint" "daisy-studio:SDS50J"
 			(at 350.52 220.65 0)
 			(effects
