File: daisy_seed.kicad_sch (KiCad schematic)
At the start: 23 parts, among them J1 SDS-50J, J4 Micro_SD_Card, J5 Conn_02x12_Odd_Even, U3 Daisy_Seed, U4 H11L1

Commit message: All the testpoints
Parts:
- renumbered J4 to J3, J1 to J4, J1 to J5, J5 to J6, J1 to J7
Other:
- note removed: "5. C_aa anti-alias cap missing. Spec calls for 1 nF C0G from each AUDIO_IN_L/R to AGND at the Seed pin. Not present. (The existing 1 nF caps C31/C33 are HF decoupling on U9's rails, not C_aa.) → Add C_aa_L (1n, between AUDIO_IN_L and GND) and C_aa_R (1n, between AUDIO_IN_R and GND), 0402/0603 C0G, near J6."
Changed lines of the file:
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@@
 		)
 	)
-	(text "  5. C_aa anti-alias cap missing.\n  Spec calls for 1 nF C0G from each AUDIO_IN_L/R to AGND at the Seed pin. Not present. (The existing 1 nF caps C31/C33 are HF decoupling on U9's rails, not\n  C_aa.) → Add C_aa_L (1n, between AUDIO_IN_L and GND) and C_aa_R (1n, between AUDIO_IN_R and GND), 0402/0603 C0G, near J6."
-		(exclude_from_sim no)
-		(at 149.098 3.302 0)
-		(effects
-			(font
-				(size 1.27 1.27)
-			)
-		)
-	)
 	(junction
 		(at 162.56 104.14)
@@
 		(dnp no)
 		(fields_autoplaced yes)
-		(property "Reference" "#PWR27"
+		(property "Reference" "#PWR027"
 			(at 224.79 166.37 0)
 			(effects
@@
 			(project "triptech"
 				(path "/55cca6a8-30da-4c13-b2f2-a01401e2b54c/75aee282-6ddd-4543-b5fc-0fc86bf548ec"
-					(reference "#PWR27")
+					(reference "#PWR027")
 					(unit 1)
 				)
@@
 		(dnp no)
 		(fields_autoplaced yes)
-		(property "Reference" "#PWR25"
+		(property "Reference" "#PWR025"
 			(at 170.18 85.09 0)
 			(effects
@@
 			(project "triptech"
 				(path "/55cca6a8-30da-4c13-b2f2-a01401e2b54c/75aee282-6ddd-4543-b5fc-0fc86bf548ec"
-					(reference "#PWR25")
+					(reference "#PWR025")
 					(unit 1)
 				)
@@
 		(dnp no)
 		(fields_autoplaced yes)
-		(property "Reference" "#PWR24"
+		(property "Reference" "#PWR024"
 			(at 147.32 49.53 0)
 			(effects
@@
 			(project ""
 				(path "/55cca6a8-30da-4c13-b2f2-a01401e2b54c/75aee282-6ddd-4543-b5fc-0fc86bf548ec"
-					(reference "#PWR24")
+					(reference "#PWR024")
 					(unit 1)
 				)
@@
 		(dnp no)
 		(fields_autoplaced yes)
-		(property "Reference" "#PWR22"
+		(property "Reference" "#PWR022"
 			(at 97.79 111.76 0)
 			(effects
@@
 			(project ""
 				(path "/55cca6a8-30da-4c13-b2f2-a01401e2b54c/75aee282-6ddd-4543-b5fc-0fc86bf548ec"
-					(reference "#PWR22")
+					(reference "#PWR022")
 					(unit 1)
 				)
@@
 		(dnp no)
 		(fields_autoplaced yes)
-		(property "Reference" "#PWR20"
+		(property "Reference" "#PWR020"
 			(at 68.58 27.94 0)
 			(effects
@@
 			(project ""
 				(path "/55cca6a8-30da-4c13-b2f2-a01401e2b54c/75aee282-6ddd-4543-b5fc-0fc86bf548ec"
-					(reference "#PWR20")
+					(reference "#PWR020")
 					(unit 1)
 				)
@@
 		(dnp no)
 		(fields_autoplaced yes)
-		(property "Reference" "#PWR28"
+		(property "Reference" "#PWR028"
 			(at 251.46 111.76 0)
 			(effects
@@
 			(project "triptech"
 				(path "/55cca6a8-30da-4c13-b2f2-a01401e2b54c/75aee282-6ddd-4543-b5fc-0fc86bf548ec"
-					(reference "#PWR28")
+					(reference "#PWR028")
 					(unit 1)
 				)
@@
 		(on_board yes)
 		(dnp no)
-		(property "Reference" "J1"
+		(property "Reference" "J4"
 			(at 158.75 78.994 0)
 			(effects
@@
 			(project ""
 				(path "/55cca6a8-30da-4c13-b2f2-a01401e2b54c/75aee282-6ddd-4543-b5fc-0fc86bf548ec"
-					(reference "J1")
+					(reference "J4")
 					(unit 1)
 				)
@@
 		(dnp no)
 		(fields_autoplaced yes)
-		(property "Reference" "#PWR26"
+		(property "Reference" "#PWR026"
 			(at 170.18 110.49 0)
 			(effects
@@
 			(project "triptech"
 				(path "/55cca6a8-30da-4c13-b2f2-a01401e2b54c/75aee282-6ddd-4543-b5fc-0fc86bf548ec"
-					(reference "#PWR26")
+					(reference "#PWR026")
 					(unit 1)
 				)
@@
 		(on_board yes)
 		(dnp no)
-		(property "Reference" "J5"
+		(property "Reference" "J6"
 			(at 215.9 119.38 0)
 			(effects
@@
 			(project ""
 				(path "/55cca6a8-30da-4c13-b2f2-a01401e2b54c/75aee282-6ddd-4543-b5fc-0fc86bf548ec"
-					(reference "J5")
+					(reference "J6")
 					(unit 1)
 				)
@@
 		(dnp no)
 		(fields_autoplaced yes)
-		(property "Reference" "J4"
+		(property "Reference" "J3"
 			(at 84.455 153.67 0)
 			(effects
@@
 			(project ""
 				(path "/55cca6a8-30da-4c13-b2f2-a01401e2b54c/75aee282-6ddd-4543-b5fc-0fc86bf548ec"
-					(reference "J4")
+					(reference "J3")
 					(unit 1)
 				)
@@
 		(dnp no)
 		(fields_autoplaced yes)
-		(property "Reference" "#PWR18"
+		(property "Reference" "#PWR018"
 			(at 40.64 123.19 0)
 			(effects
@@
 			(project ""
 				(path "/55cca6a8-30da-4c13-b2f2-a01401e2b54c/75aee282-6ddd-4543-b5fc-0fc86bf548ec"
-					(reference "#PWR18")
+					(reference "#PWR018")
 					(unit 1)
 				)
@@
 		(dnp no)
 		(fields_autoplaced yes)
-		(property "Reference" "#PWR21"
+		(property "Reference" "#PWR021"
 			(at 76.2 27.94 0)
 			(effects
@@
 			(project ""
 				(path "/55cca6a8-30da-4c13-b2f2-a01401e2b54c/75aee282-6ddd-4543-b5fc-0fc86bf548ec"
-					(reference "#PWR21")
+					(reference "#PWR021")
 					(unit 1)
 				)
@@
 		(on_board yes)
 		(dnp no)
-		(property "Reference" "J1"
+		(property "Reference" "J5"
 			(at 158.75 105.918 0)
 			(effects
@@
 			(project "triptech"
 				(path "/55cca6a8-30da-4c13-b2f2-a01401e2b54c/75aee282-6ddd-4543-b5fc-0fc86bf548ec"
-					(reference "J1")
+					(reference "J5")
 					(unit 1)
 				)
@@
 		(on_board yes)
 		(dnp no)
-		(property "Reference" "J1"
+		(property "Reference" "J7"
 			(at 242.062 96.012 0)
 			(effects
@@
 			(project "triptech"
 				(path "/55cca6a8-30da-4c13-b2f2-a01401e2b54c/75aee282-6ddd-4543-b5fc-0fc86bf548ec"
-					(reference "J1")
+					(reference "J7")
 					(unit 1)
 				)
@@
 		(dnp no)
 		(fields_autoplaced yes)
-		(property "Reference" "#PWR19"
+		(property "Reference" "#PWR019"
 			(at 60.96 27.94 0)
 			(effects
@@
 			(project ""
 				(path "/55cca6a8-30da-4c13-b2f2-a01401e2b54c/75aee282-6ddd-4543-b5fc-0fc86bf548ec"
-					(reference "#PWR19")
+					(reference "#PWR019")
 					(unit 1)
 				)
@@
 		(dnp no)
 		(fields_autoplaced yes)
-		(property "Reference" "#PWR23"
+		(property "Reference" "#PWR023"
 			(at 104.14 200.66 0)
 			(effects
@@
 			(project "triptech"
 				(path "/55cca6a8-30da-4c13-b2f2-a01401e2b54c/75aee282-6ddd-4543-b5fc-0fc86bf548ec"
-					(reference "#PWR23")
+					(reference "#PWR023")
 					(unit 1)
 				)
