File: daisy_seed.kicad_sch (KiCad schematic)
At the start: 23 parts, among them J10 SDS-50J, J11 Conn_02x12_Odd_Even, J14 Micro_SD_Card_Det2, J7 SDS-50J, J9 SDS-50J, U8 H11L1, U9 Daisy_Seed

Commit message: fix header
Parts:
- J11: value Conn_02x12_Odd_Even -> Conn_02x14_Odd_Even
Changed lines of the file:
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@@
 			)
 		)
-		(property "Value" "Conn_02x12_Odd_Even"
+		(property "Value" "Conn_02x14_Odd_Even"
 			(at 215.392 118.364 0)
 			(effects
