File: daisy-studio.kicad_pcb (KiCad board)
At the start: 4 copper layers, 278.3 x 56.7 mm, 149 parts, among them J1 NCJ6FA-H-0, J10 SDS-50J, J11 Conn_02x12_Odd_Even, J12 Conn_02x02_Odd_Even, J13 Barrel_Jack_MountingPin, J14 Micro_SD_Card_Det2, J2 NCJ6FA-H-0, J3 Conn_02x10_Odd_Even, J4 NCJ6FA-H-0, J5 Conn_02x10_Odd_Even, J6 NCJ6FA-H-0, J7 SDS-50J, J9 SDS-50J, Q1 MMBT3904, Q2 MMBT3906, Q3 MMBT3906, Q4 MMBT3904, Q5 DMP3056L-13, SW1 Power, U1 THAT1646, U10 TPS54302, U2 THAT1646, U3 OPA1656ID, U4 THAT1246, U5 THAT1246, U6 OPA1656ID, U7 LM2903, U8 H11L1, U9 Daisy_Seed

Commit message: Rev2b - fix LEDs
Parts:
- moved D9 13.7 mm to (54.3, 60.0)
- moved D10 13.6 mm to (54.3, 73.6)
Routing:
- net CLIP_LED_K_R: track 123.3 -> 145.7 mm, vias 2 -> 1
- net CLIP_LED_A_R: track 45.5 -> 66.7 mm
- net CLIP_LED_A_L: track 44.5 -> 59.6 mm
- net CLIP_LED_K_L: track 94.9 -> 109.9 mm
- net IN_WIPER_R: track 62.4 -> 57.4 mm
- net GND: track 229.6 -> 228.6 mm, vias 2242 -> 2193
- net Net-(D3-K): track 56.9 -> 56.0 mm
Other:
- board text added: "Gain/Clip Daisy-Studio Rev2b 29 Apr 2026 Rasheed Abdul-Aziz"
- board text added: "Main Daisy-Studio Rev2b 29 Apr 2026 Rasheed Abdul-Aziz"
- board text removed: "Gain/Clip Daisy-Studio Rev2 29 Apr 2026 Rasheed Abdul-Aziz"
- board text removed: "Main Daisy-Studio Rev2 29 Apr 2026 Rasheed Abdul-Aziz"
