File: daughter-board/daughter-board.kicad_sch (KiCad schematic)
At the start: 8 parts, among them J5 Conn_02x10_Odd_Even

Commit message: split finished up without finalizing the daughterboard
Other:
- title: (none) -> Daisy-Studio Daughterboard
Changed lines of the file:
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@@
 	(generator_version "9.0")
 	(paper "A4")
+	(title_block
+		(title "Daisy-Studio Daughterboard")
+		(rev "2c")
+	)
 	(text "Output\n"
 		(exclude_from_sim no)
