File: main-board/audio_output.kicad_sch (KiCad schematic)
At the start: 33 parts, among them J1 NCJ6FA-H-0, J2 NCJ6FA-H-0, U1 THAT1646, U2 THAT1646, U3 OPA1656ID

Commit message: swap and label rv8/7 so they lay out clearly
fixes #21
Parts:
- RV2: Label (none) -> OGT_L
- RV4: Label (none) -> OGT_R
Changed lines of the file:
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@@
+			)
+		)
+		(property "Label" "OGT_L"
+			(at 107.95 41.91 90)
+			(effects
+				(font
+					(size 1.27 1.27)
+				)
+				(hide yes)
 			)
 		)
@@
 			(effects
 				(font
+					(size 1.27 1.27)
+				)
+				(hide yes)
+			)
+		)
+		(property "Label" "OGT_R"
+			(at 107.95 101.6 90)
+			(effects
+				(font
